Commit message: correct error in robot_core

File: description/robot_core.xacro (robot description, xacro)
@@ -1,14 +1,14 @@
 <?xml version="1.0"?>
-<robot xmlns:xacro="http://www.ros.org/wiki/xacro">
-    <material name="white"/>
+<robot>
+    <material name="white">
         <color rgba="1 1 1 1"/>
     </material>
-    <material name="orange"/>
+    <material name="orange">
         <color rgba="1 0.3 0.1 1"/>
     </material>
-    <material name="blue"/>
+    <material name="blue">
         <color rgba="0.2 0.2 1 1"/>
     </material>
-    <material name="black"/>
+    <material name="black">
         <color rgba="0 0 0 1"/>
     </material>

Commit message: correct error in xacro

File: description/robot_core.xacro (robot description, xacro)
@@ -24,5 +24,5 @@
             <origin xyz="0.15 0 0.075"/>
             <geometry>
-                <box size="0.3 0.3 015"/>
+                <box size="0.3 0.3 0.15"/>
             </geometry>
             <material name="blue"/>

Commit message: add wheels

File: description/robot_core.xacro (robot description, xacro)
@@ -13,6 +13,8 @@
         <color rgba="0 0 0 1"/>
     </material>
+    <!-- BASE LINK-->
     <link name="base_link">
     </link>
+    <!--CHASSIS LINK-->
     <joint name="chassis_joint" type="fixed">
         <parent link="base_link"/>
@@ -29,3 +31,33 @@
         </visual>
     </link>
+   <!-- LEFT WHEEL LINK -->
+    <joint name="left_wheel_joint" type="cntinuous">
+            <parent link="base_link"/>
+            <child link="left_wheel"/>
+            <origin xyz="0 0.175 0" rpy="-${pi/2} 0 0"/>
+            <axis xyz="0 0 1"/>
+    </joint>
+    <link name="left_wheel">
+        <visual>
+            <geometry>
+                <cylinder radius="0.05" length="0.04"/>
+            </geometry>
+            <material name="white"/>
+        </visual>
+    </link>
+    <!-- RIGHT WHEEL LINK -->
+    <joint name="right_wheel_joint" type="cntinuous">
+            <parent link="base_link"/>
+            <child link="right_wheel"/>
+            <origin xyz="0 -0.175 0" rpy="${pi/2} 0 0"/>
+            <axis xyz="0 0 -1"/>
+    </joint>
+    <link name="right_wheel">
+        <visual>
+            <geometry>
+                <cylinder radius="0.05" length="0.04"/>
+            </geometry>
+            <material name="white"/>
+        </visual>
+    </link>
 </robot>

Commit message: xacro changes

File: description/robot_core.xacro (robot description, xacro)
@@ -32,5 +32,5 @@
     </link>
    <!-- LEFT WHEEL LINK -->
-    <joint name="left_wheel_joint" type="cntinuous">
+    <joint name="left_wheel_joint" type="continuous">
             <parent link="base_link"/>
             <child link="left_wheel"/>
@@ -47,5 +47,5 @@
     </link>
     <!-- RIGHT WHEEL LINK -->
-    <joint name="right_wheel_joint" type="cntinuous">
+    <joint name="right_wheel_joint" type="continuous">
             <parent link="base_link"/>
             <child link="right_wheel"/>

Commit message: add collision

File: description/robot_core.xacro (robot description, xacro)
@@ -30,4 +30,10 @@
             <material name="blue"/>
         </visual>
+        <collision>
+            <origin xyz="0.15 0 0.075"/>
+            <geometry>
+                <box size="0.3 0.3 0.15"/>
+            </geometry>
+        </collision>
     </link>
    <!-- LEFT WHEEL LINK -->
@@ -45,4 +51,9 @@
             <material name="white"/>
         </visual>
+        <collision>
+            <geometry>
+                <cylinder radius="0.05" length="0.04"/>
+            </geometry>
+        </collision>
     </link>
     <!-- RIGHT WHEEL LINK -->
@@ -60,4 +71,28 @@
             <material name="white"/>
         </visual>
+        <collision>
+            <geometry>
+                <cylinder radius="0.05" length="0.04"/>
+            </geometry>
+        </collision>
+    </link>
+    <!-- CASTER WHEEL LINK-->
+    <joint name="caster_wheel_joint" type="fixed">
+        <parent link="chassis"/>
+        <child link="caster_wheel"/>
+        <origin xyz="0.24 0 0"/>
+    </joint>
+    <link name="caster_wheel">
+        <visual>
+            <geometry>
+                <sphere radius="0.05"/>
+            </geometry>
+            <material name="white"/>
+        </visual>
+         <collision>
+            <geometry>
+                <sphere radius="0.05"/>
+            </geometry>
+         </collision>
     </link>
 </robot>

Commit message: add new inertial_macros

File: description/robot_core.xacro (robot description, xacro)
@@ -1,4 +1,5 @@
 <?xml version="1.0"?>
 <robot>
+    <xacro:include filename="inertial_macros.xacro"/>
     <material name="white">
         <color rgba="1 1 1 1"/>
@@ -36,4 +37,7 @@
             </geometry>
         </collision>
+        <xacro:inertial_box mass="0.5" x="0.3" y="0.3" z="0.15">
+            <origin xyz="0.15 0 0.075" rpy="0 0 0"/>
+        </xacro:inertial_box>
     </link>
    <!-- LEFT WHEEL LINK -->

Commit message: add inf lidar file

File: description/robot_core.xacro (robot description, xacro)
@@ -14,4 +14,7 @@
     <material name="black">
         <color rgba="0 0 0 1"/>
+    </material>
+     <material name="red">
+        <color rgba="1 0 0 1"/>
     </material>
     <!-- BASE LINK-->
