Commit message: correct camera file

File: description/camera.xacro (robot description, xacro)
@@ -13,5 +13,5 @@
             <material name="red"/>
         </visual>
-        <collision>
+        <!--<collision>
             <geometry>
                 <box size="0.01 0.03 0.03"/>
@@ -21,4 +21,5 @@
             <origin xyz="0 0 0" rpy="0 0 0"/>
         </xacro:inertial_box>
+        /-->
     </link>
      <joint name="camera_optical_joint" type="fixed">
@@ -30,30 +31,24 @@
     <gazebo reference="camera_link">
         <material>Gazebo/Red</material>
-    <!-- <sensor name="laser" type="ray">
+        <sensor name="camera" type="ray">
             <pose> 0 0 0 0 0 0 </pose>
             <visualize>true</visualize>
             <update_rate>10</update_rate>
-            <ray>
-                <scan>
-                    <horizontal>
-                        <samples>360</samples>
-                        <min_angle>-3.14</min_angle>
-                        <max_angle>3.14</max_angle>
-                    </horizontal>
-                </scan>
-                <range>
-                    <min>0.3</min>
-                    <max>12</max>
-                </range>
-            </ray>
-            <plugin name="laser_controller" filename="libgazebo_ros_ray_sensor.so">
-                <ros>
-                    <argument>~/out:=scan</argument>
-                </ros>
-                <output_type>sensor_msgs/LaserScan</output_type>
-                <frame_name>laser_frame</frame_name>
+            <camera>
+                <horizontal_fov>1.089</horizontal_fov>
+                <image>
+                    <format>R8G8B8</format>
+                    <width>640</width>
+                    <height>480</height>
+                </image>
+                <clip>
+                    <near>0.05</near>
+                    <far>8.0</far>
+                </clip>
+            </camera>
+            <plugin name="camera_controller" filename="libgazebo_ros_camera.so">
+                <frame_name>camera_link_optical</frame_name>
             </plugin>
         </sensor>
-    /-->
     </gazebo>
 </robot>

Commit message: correct camera file

File: description/camera.xacro (robot description, xacro)
@@ -26,10 +26,10 @@
         <parent link="camera_link"/>
         <child link="camera_link_optical"/>
-        <origin xyz="0 0 0" rpy="${-pi/2} 0 ${pi/2}"/>
+        <origin xyz="0 0 0" rpy="${-pi/2} 0 ${-pi/2}"/>
     </joint>
     <link name="camera_link_optical"></link>
     <gazebo reference="camera_link">
         <material>Gazebo/Red</material>
-        <sensor name="camera" type="ray">
+        <sensor name="camera" type="camera">
             <pose> 0 0 0 0 0 0 </pose>
             <visualize>true</visualize>
