Commit message: complit lidar files

File: description/lidar.xacro (robot description, xacro)
@@ -18,7 +18,35 @@
             </geometry>
         </collision>
-        <xacro:inertial_cylinder mass="0.1"  radius="0.05" length="0.04">
+        <xacro:inertial_cylinder mass="0.1" length="0.04" radius="0.05">
             <origin xyz="0 0 0" rpy="0 0 0"/>
-        </xacro:inertial_cylinder >
+        </xacro:inertial_cylinder>
     </link>
+    <gazebo reference="laser_frame">
+        <material>Gazebo/Red</material>
+        <sensor name="laser" type="ray">
+            <pose> 0 0 0 0 0 0 </pose>
+            <visualize>true</visualize>
+            <update_rate>10</update_rate>
+            <ray>
+                <scan>
+                    <horizontal>
+                        <samples>360</samples>
+                        <min_angle>-3.14</min_angle>
+                        <max_angle>3.14</max_angle>
+                    </horizontal>
+                </scan>
+                <range>
+                    <min>0.3</min>
+                    <max>12</max>
+                </range>
+            </ray>
+            <plugin name="laser_controller" filename="libgazebo_ros_ray_sensor.so">
+                <ros>
+                    <argument>~/out:=scan</argument>
+                </ros>
+                <output_type>sensor_msgs/LaserScan</output_type>
+                <frame_name>laser_frame</frame_name>
+            </plugin>
+        </sensor>
+    </gazebo>
 </robot>

Commit message: add xacro file 2 cart

File: description/lidar.xacro (robot description, xacro)
@@ -22,31 +22,3 @@
         </xacro:inertial_cylinder>
     </link>
-    <gazebo reference="laser_frame">
-        <material>Gazebo/Red</material>
-        <sensor name="laser" type="ray">
-            <pose> 0 0 0 0 0 0 </pose>
-            <visualize>true</visualize>
-            <update_rate>10</update_rate>
-            <ray>
-                <scan>
-                    <horizontal>
-                        <samples>360</samples>
-                        <min_angle>-3.14</min_angle>
-                        <max_angle>3.14</max_angle>
-                    </horizontal>
-                </scan>
-                <range>
-                    <min>0.3</min>
-                    <max>12</max>
-                </range>
-            </ray>
-            <plugin name="laser_controller" filename="libgazebo_ros_ray_sensor.so">
-                <ros>
-                    <argument>~/out:=scan</argument>
-                </ros>
-                <output_type>sensor_msgs/LaserScan</output_type>
-                <frame_name>laser_frame</frame_name>
-            </plugin>
-        </sensor>
-    </gazebo>
 </robot>

File: description/robot.urdf.xacro (robot description, xacro)
@@ -2,4 +2,5 @@
 <robot xmlns:xacro="http://www.ros.org/wiki/xacro"  name="robot">
     <xacro:include filename = "robot_core.xacro"/>
+    <xacro:include filename = "robot_core_2.xacro"/>
     <xacro:include filename = "gazebo_control.xacro"/>
     <xacro:include filename = "lidar.xacro"/>

File: description/robot_core.xacro (robot description, xacro)
@@ -2,5 +2,6 @@
 <robot xmlns:xacro="http://www.ros.org/wiki/xacro">
     <xacro:include filename="inertial_macros.xacro"/>
-    <!--material color -->
+    <!-- ######################################################################## /-->
+    <!--material color /-->
     <material name="white">
         <color rgba="1 1 1 1"/>
@@ -15,11 +16,13 @@
         <color rgba="0 0 0 1"/>
     </material>
-     <material name="red">
+    <material name="red">
         <color rgba="1 0 0 1"/>
     </material>
-    <!-- BASE LINK-->
+    <!-- BASE LINK/-->
     <link name="base_link">
     </link>
-    <!--CHASSIS LINK-->
+    <!-- BASE LINK-->
+    <!-- ########################################################################-->
+    <!--CHASSIS LINK/-->
     <joint name="chassis_joint" type="fixed">
         <parent link="base_link"/>
@@ -48,9 +51,11 @@
         <material>Gazebo/Blue</material>
     </gazebo>
-   <!-- LEFT WHEEL LINK -->
+    <!--CHASSIS LINK-->
+    <!-- ######################################################################## -->
+    <!-- LEFT WHEEL LINK -->
     <joint name="left_wheel_joint" type="continuous">
             <parent link="base_link"/>
             <child link="left_wheel"/>
-            <origin xyz="0 0.175 0" rpy="-${pi/2} 0 0"/>
+            <origin xyz="0.14 0.175 0" rpy="-${pi/2} 0 0"/>
             <axis xyz="0 0 1"/>
     </joint>
@@ -74,9 +79,11 @@
         <material>Gazebo/White</material>
     </gazebo>
+    <!-- LEFT WHEEL LINK -->
+    <!-- ######################################################################## -->
     <!-- RIGHT WHEEL LINK -->
     <joint name="right_wheel_joint" type="continuous">
             <parent link="base_link"/>
             <child link="right_wheel"/>
-            <origin xyz="0 -0.175 0" rpy="${pi/2} 0 0"/>
+            <origin xyz="0.14 -0.175 0" rpy="${pi/2} 0 0"/>
             <axis xyz="0 0 -1"/>
     </joint>
@@ -100,9 +107,11 @@
         <material>Gazebo/White</material>
     </gazebo>
+     <!-- RIGHT WHEEL LINK -->
+    <!-- ######################################################################## -->
     <!-- CASTER WHEEL LINK-->
     <joint name="caster_wheel_joint" type="fixed">
         <parent link="chassis"/>
         <child link="caster_wheel"/>
-        <origin xyz="0.24 0 0"/>
+        <origin xyz="0.08 0 0"/>
     </joint>
     <link name="caster_wheel">
@@ -113,10 +122,10 @@
             <material name="white"/>
         </visual>
-         <collision>
+        <collision>
             <geometry>
                 <sphere radius="0.05"/>
             </geometry>
-         </collision>
-         <xacro:inertial_sphere mass="0.1" radius="0.05" >
+        </collision>
+        <xacro:inertial_sphere mass="0.1" radius="0.05" >
             <origin xyz="0 0 0" rpy="0 0 0"/>
         </xacro:inertial_sphere>
@@ -127,3 +136,4 @@
         <mu2 value = "0.001"/>
     </gazebo>
+    <!-- CASTER WHEEL LINK-->
 </robot>
