Commit message: create new files-py

File: description/pendulum.xacro (robot description, xacro)
@@ -23,15 +23,15 @@
                 </geometry>
                 <material name="black"/>
-                <origin rpy="0 0 0" xyz="0 0 0.15"/>
+                <origin rpy="0 0 0" xyz="0 0 0.3"/>
                 </visual>
             </link>
             <joint name="pole_joint" type="revolute">
-                <parent link="conector_pole"/>
+                <parent link="chassis"/>
                 <child link="pole"/>
-                <origin xyz="0 0 0" rpy="0 0 0.15"/>
-                <axis xyz="0 1 0"/>
-                <limit effort="1000.0" lower="-1.57075" upper="1.57075" velocity="1.0"/>
+                <origin xyz="0.15 0 0" rpy="0 0 -0.15"/>
+                <axis xyz="0 1.0 0"/>
+                <limit effort="1000.0" lower="-0.57075" upper="0.57075" velocity="1.0"/>
             </joint>
-            <!--link name="pole_mass">
+            <link name="pole_mass">
                 <visual>
                 <geometry>
@@ -47,10 +47,10 @@
                 <parent link="pole"/>
                 <child link="pole_mass"/>
-            </joint-->
+            </joint>
             <gazebo reference = "pole">
-                <material>Gazebo/Black</material>
+                <material>Gazebo/black</material>
             </gazebo>
             <gazebo reference = "pole_mass">
-                <material>Gazebo/Blue</material>
+                <material>Gazebo/blue</material>
             </gazebo>
         <!--Pendulum/-->

File: description/robot_core.xacro (robot description, xacro)
@@ -19,4 +19,9 @@
         <color rgba="1 0 0 1"/>
     </material>
+    <gazebo>
+        <plugin filename="libgazebo_ros_control.so" name="gazebo_ros_control">
+          <robotSimType>sr_gazebo_sim/SrGazeboHWSim</robotSimType>
+        </plugin>
+      </gazebo>
     <!-- BASE LINK/-->
     <link name="base_link">

Commit message: version 24.10

File: description/pendulum.xacro (robot description, xacro)
@@ -4,4 +4,9 @@
         <!--Pendulum-->
         <link name="conector_pole">
+            <inertial>
+                <origin xyz="0.0 0.0 0.0" rpy="0.0 0.0 0.0"/>
+                <mass value="0.01"/>
+                <inertia ixx="0.0" ixy="0.0" ixz="0.0" iyy="0.0" iyz="0.0" izz="0.0"/>
+            </inertial>
             <visual>
                 <geometry>
@@ -11,4 +16,9 @@
                 <origin rpy="0 0 0" xyz="0 0 0"/>
             </visual>
+            <collision>
+                <geometry>
+                    <box size="0.02 0.02 0.02"/>
+                </geometry>
+            </collision>
         </link>
         <joint name="conector_pole_joint" type="fixed">
@@ -18,4 +28,9 @@
         </joint>
             <link name="pole">
+                <inertial>
+                    <origin xyz="0.0 0.0 0.0" rpy="0.0 0.0 0.0"/>
+                    <mass value="0.01"/>
+                    <inertia ixx="0.0" ixy="0.0" ixz="0.0" iyy="0.0" iyz="0.0" izz="0.0"/>
+                </inertial>
                 <visual>
                 <geometry>
@@ -23,15 +38,25 @@
                 </geometry>
                 <material name="black"/>
-                <origin rpy="0 0 0" xyz="0 0 0.3"/>
+                <origin rpy="0 0 0" xyz="0 0 0"/>
                 </visual>
+                <collision>
+                <geometry>
+                    <cylinder length="0.3" radius="0.01"/>
+                </geometry>
+            </collision>
             </link>
             <joint name="pole_joint" type="revolute">
-                <parent link="chassis"/>
+                <parent link="conector_pole"/>
                 <child link="pole"/>
-                <origin xyz="0.15 0 0" rpy="0 0 -0.15"/>
+                <origin xyz="0 0 0.3" rpy="0 0 0"/>
                 <axis xyz="0 1.0 0"/>
                 <limit effort="1000.0" lower="-0.57075" upper="0.57075" velocity="1.0"/>
             </joint>
             <link name="pole_mass">
+                <inertial>
+                    <origin xyz="0.0 0.0 0.0" rpy="0.0 0.0 0.0"/>
+                    <mass value="0.01"/>
+                    <inertia ixx="0.0" ixy="0.0" ixz="0.0" iyy="0.0" iyz="0.0" izz="0.0"/>
+                </inertial>
                 <visual>
                 <geometry>

Commit message: version 24.10 12:15

File: description/pendulum.xacro (robot description, xacro)
@@ -21,4 +21,7 @@
                 </geometry>
             </collision>
+            <xacro:inertial_box mass="0.01" x="0.02" y="0.02" z="0.02">
+                <origin xyz="0 0 0" rpy="0 0 0"/>
+            </xacro:inertial_box>
         </link>
         <joint name="conector_pole_joint" type="fixed">
@@ -27,11 +30,6 @@
             <origin xyz="0.15 0 0.15" />
         </joint>
-            <link name="pole">
-                <inertial>
-                    <origin xyz="0.0 0.0 0.0" rpy="0.0 0.0 0.0"/>
-                    <mass value="0.01"/>
-                    <inertia ixx="0.0" ixy="0.0" ixz="0.0" iyy="0.0" iyz="0.0" izz="0.0"/>
-                </inertial>
-                <visual>
+        <link name="pole">
+            <visual>
                 <geometry>
                     <cylinder length="0.3" radius="0.01"/>
@@ -39,19 +37,22 @@
                 <material name="black"/>
                 <origin rpy="0 0 0" xyz="0 0 0"/>
-                </visual>
-                <collision>
+            </visual>
+            <collision>
                 <geometry>
                     <cylinder length="0.3" radius="0.01"/>
                 </geometry>
             </collision>
-            </link>
-            <joint name="pole_joint" type="revolute">
-                <parent link="conector_pole"/>
-                <child link="pole"/>
-                <origin xyz="0 0 0.3" rpy="0 0 0"/>
-                <axis xyz="0 1.0 0"/>
-                <limit effort="1000.0" lower="-0.57075" upper="0.57075" velocity="1.0"/>
-            </joint>
-            <link name="pole_mass">
+            <xacro:inertial_cylinder mass="0.05"  radius="0.01" length="0.03">
+                <origin xyz="0 0 0" rpy="0 0 0"/>
+            </xacro:inertial_cylinder >
+        </link>
+        <joint name="pole_joint" type="revolute">
+            <parent link="conector_pole"/>
+            <child link="pole"/>
+            <origin xyz="0 0 0.3" rpy="0 0 0"/>
+            <axis xyz="0 1.0 0"/>
+            <limit effort="1000.0" lower="-0.57075" upper="0.57075" velocity="1.0"/>
+        </joint>
+            <!--link name="pole_mass">
                 <inertial>
                     <origin xyz="0.0 0.0 0.0" rpy="0.0 0.0 0.0"/>
@@ -72,11 +73,14 @@
                 <parent link="pole"/>
                 <child link="pole_mass"/>
-            </joint>
+            </joint-->
             <gazebo reference = "pole">
                 <material>Gazebo/black</material>
             </gazebo>
-            <gazebo reference = "pole_mass">
+            <gazebo reference = "conector_pole">
+                <material>Gazebo/white</material>
+            </gazebo>
+            <!--gazebo reference = "pole_mass">
                 <material>Gazebo/blue</material>
-            </gazebo>
+            </gazebo-->
         <!--Pendulum/-->
 </robot>
