Commit message: version 24.10 11:50

File: description/robot_core_2.xacro (robot description, xacro)
@@ -16,4 +16,11 @@
             <material name="red"/>
         </visual>
+        <collision>
+            <origin xyz="0.0 0.0 0.0" rpy="0.0 0.0 0.0"/>
+            <box size="0.01 0.03 0.03"/>
+        </collision>
+        <xacro:inertial_box mass="0.01" x="0.01" y="0.03" z="0.03">
+            <origin xyz="0.15 0 0.075" rpy="0 0 0"/>
+        </xacro:inertial_box>
     </link>
     <gazebo reference="conector_link">

Commit message: version 24.10 12:00

File: description/robot_core_2.xacro (robot description, xacro)
@@ -43,4 +43,11 @@
             <material name="red"/>
         </visual>
+        <collision>
+            <origin xyz="0.0 0.0 0.0" rpy="0.0 0.0 0.0"/>
+            <box size="0.3 0.02 0.02"/>
+        </collision>
+        <xacro:inertial_box mass="0.1" x="0.3" y="0.02" z="0.02">
+            <origin xyz="0 0 0" rpy="0 0 0"/>
+        </xacro:inertial_box>
     </link>
     <gazebo reference="element1_link">
@@ -64,4 +71,11 @@
                 <material name="red"/>
             </visual>
+            <collision>
+                <origin xyz="0.0 0.0 0.0" rpy="0.0 0.0 0.0"/>
+                <box size="0.15 0.02 0.02"/>
+            </collision>
+            <xacro:inertial_box mass="0.01" x="0.15" y="0.02" z="0.02">
+                <origin xyz="0 0 0" rpy="0 0 0"/>
+            </xacro:inertial_box>
         </link>
         <gazebo reference="element2_link">
@@ -82,4 +96,11 @@
                 <material name="red"/>
             </visual>
+            <collision>
+                <origin xyz="0.0 0.0 0.0" rpy="0.0 0.0 0.0"/>
+                <box size="0.01 0.03 0.03"/>
+            </collision>
+            <xacro:inertial_box mass="0.01" x="0.01" y="0.03" z="0.03">
+                <origin xyz="0 0 0" rpy="0 0 0"/>
+            </xacro:inertial_box>
         </link>
         <gazebo reference="conector_2_link">

Commit message: version 24.10 12:10

File: description/robot_core_2.xacro (robot description, xacro)
@@ -2,5 +2,4 @@
 <robot xmlns:xacro="http://www.ros.org/wiki/xacro">
     <xacro:include filename="inertial_macros.xacro"/>
-    <!-- ######################################################################## -->
     <!--Connector-->
     <joint name="conector_joint" type="fixed">
@@ -27,6 +26,4 @@
         <material>Gazebo/Red</material>
     </gazebo>
-    <!--Connector/-->
-    <!-- ######################################################################## -->
     <!--element1-->
     <joint name="element1_joint" type="fixed">
@@ -54,5 +51,4 @@
         <material>Gazebo/Red</material>
     </gazebo>
-    <!--element1/-->
     <!--element2/-->
         <joint name="element2_joint" type="fixed">
@@ -82,5 +78,4 @@
             <material>Gazebo/Red</material>
         </gazebo>
-    <!--element2/-->
     <!--conector_2/-->
         <joint name="conector_2_joint" type="fixed">
@@ -107,5 +102,4 @@
             <material>Gazebo/Red</material>
         </gazebo>
-    <!--conector_2/-->
     <!--CHASSIS LINK 2-->
         <joint name="chassis_2_joint" type="fixed">
@@ -116,5 +110,5 @@
         <link name="chassis_2">
             <visual>
-                <origin xyz="-0.15 0 0.075"/>
+                <origin xyz="0 0 0"/>
                 <geometry>
                     <box size="0.3 0.3 0.15"/>
@@ -123,5 +117,5 @@
             </visual>
             <collision>
-                <origin xyz="0.15 0 0.075"/>
+                <origin xyz="0 0 0"/>
                 <geometry>
                     <box size="0.3 0.3 0.15"/>
@@ -129,5 +123,5 @@
             </collision>
             <xacro:inertial_box mass="0.5" x="0.3" y="0.3" z="0.15">
-                <origin xyz="0.15 0 0.075" rpy="0 0 0"/>
+                <origin xyz="0 0 0" rpy="0 0 0"/>
             </xacro:inertial_box>
         </link>
@@ -135,5 +129,4 @@
             <material>Gazebo/Blue</material>
         </gazebo>
-    <!--CHASSIS LINK 2-->
     <!-- LEFT WHEEL LINK 2-->
         <joint name="left_wheel_2_joint" type="fixed">
@@ -162,5 +155,4 @@
             <material>Gazebo/White</material>
         </gazebo>
-    <!-- LEFT WHEEL LINK 2-->
     <!-- RIGHT WHEEL LINK 2-->
         <joint name="right_wheel_2_joint" type="continuous">
@@ -189,5 +181,4 @@
             <material>Gazebo/White</material>
         </gazebo>
-    <!-- RIGHT WHEEL LINK 2-->
     <!-- CASTER WHEEL LINK-->
         <joint name="caster_wheel_2_joint" type="fixed">
@@ -217,4 +208,3 @@
             <mu2 value = "0.001"/>
         </gazebo>
-    <!-- CASTER WHEEL LINK2-->
 </robot>

Commit message: version 16_00

File: description/robot_core_2.xacro (robot description, xacro)
@@ -16,5 +16,4 @@
         </visual>
         <collision>
-            <origin xyz="0.0 0.0 0.0" rpy="0.0 0.0 0.0"/>
             <box size="0.01 0.03 0.03"/>
         </collision>
@@ -41,5 +40,4 @@
         </visual>
         <collision>
-            <origin xyz="0.0 0.0 0.0" rpy="0.0 0.0 0.0"/>
             <box size="0.3 0.02 0.02"/>
         </collision>
@@ -52,5 +50,5 @@
     </gazebo>
     <!--element2/-->
-        <joint name="element2_joint" type="fixed">
+        <joint name="element2_joint" type="revolute">
             <parent link="element1_link"/>
             <child link="element2_link"/>
