Commit message: add pendulum file

File: description/gazebo_control.xacro (robot description, xacro)
@@ -6,4 +6,6 @@
                 <left_joint>left_wheel_joint</left_joint>
                 <right_joint>right_wheel_joint</right_joint>
+                <!--left_joint>left_wheel_2_joint</left_joint>
+                <right_joint>right_wheel_2_joint</right_joint-->
                 <wheel_separation>0.35</wheel_separation>
                 <wheel_diameter>0.1</wheel_diameter>

File: description/lidar.xacro (robot description, xacro)
@@ -4,5 +4,5 @@
         <parent link="chassis"/>
         <child link="laser_frame"/>
-        <origin xyz="0.1 0 0.175" rpy="0 0 0"/>
+        <origin xyz="0.122 0 0.212" rpy="0 0 0"/>
     </joint>
     <link name="laser_frame">
@@ -11,5 +11,12 @@
                 <cylinder radius="0.05" length="0.04"/>
             </geometry>
-            <material name="red"/>
+            <material name="black"/>
+        </visual>
+        <visual>
+            <origin xyz="0 0 -0.05"/>
+            <geometry>
+                <cylinder radius="0.01" length="0.1"/>
+            </geometry>
+            <material name="black"/>
         </visual>
         <collision>
@@ -22,3 +29,31 @@
         </xacro:inertial_cylinder>
     </link>
+    <gazebo reference="laser_frame">
+        <material>Gazebo/Black</material>
+        <sensor name="laser" type="ray">
+            <pose> 0 0 0 0 0 0 </pose>
+            <visualize>false</visualize>
+            <update_rate>10</update_rate>
+            <ray>
+                <scan>
+                    <horizontal>
+                        <samples>360</samples>
+                        <min_angle>-3.14</min_angle>
+                        <max_angle>3.14</max_angle>
+                    </horizontal>
+                </scan>
+                <range>
+                    <min>0.3</min>
+                    <max>12</max>
+                </range>
+            </ray>
+            <plugin name="laser_controller" filename="libgazebo_ros_ray_sensor.so">
+                <ros>
+                    <argument>~/out:=scan</argument>
+                </ros>
+                <output_type>sensor_msgs/LaserScan</output_type>
+                <frame_name>laser_frame</frame_name>
+            </plugin>
+        </sensor>
+    </gazebo>
 </robot>

File: description/robot.urdf.xacro (robot description, xacro)
@@ -2,7 +2,8 @@
 <robot xmlns:xacro="http://www.ros.org/wiki/xacro"  name="robot">
     <xacro:include filename = "robot_core.xacro"/>
-    <xacro:include filename = "robot_core_2.xacro"/>
+    <!--xacro:include filename = "robot_core_2.xacro"/-->
     <xacro:include filename = "gazebo_control.xacro"/>
-    <xacro:include filename = "lidar.xacro"/>
+    <xacro:include filename = "pendulum.xacro"/>
+    <!--xacro:include filename = "lidar.xacro"/-->
     <xacro:include filename = "camera.xacro"/>
 </robot>

File: description/robot_core_2.xacro (robot description, xacro)
@@ -46,4 +46,5 @@
             <child link="element2_link"/>
             <axis xyz="0 0 1"/>
+            <!--limit effort="1000.0" lower="0.0" upper="0.548" velocity="0.5"/-->
             <origin xyz="-0.15 0 0" rpy="0 0 0"/>
         </joint>
@@ -53,4 +54,5 @@
                     <box size="0.15 0.02 0.02"/>
                 </geometry>
+                <origin rpy="1.57074 0 0" xyz="0.075 0 0"/>>
                 <material name="red"/>
             </visual>
@@ -133,59 +135,4 @@
         </gazebo>
     <!-- LEFT WHEEL LINK 2-->
-    <!--Pendulum-->
-    <link name="conector_pole">
-        <visual>
-        <geometry>
-            <box size="0.2 0.2 0.2"/>
-        </geometry>
-        <material name="black"/>
-        <origin rpy="0 0 0" xyz="0.0 0 -0.1"/>
-        </visual>
-    </link>
-    <joint name="conector_pole_joint" type="revolute">
-        <origin xyz="-0.15 0 0.36" rpy="0 0 0"/>
-        <axis xyz="0 1 0"/>
-        <parent link="chassis_2"/>
-        <child link="conector_pole"/>
-        <limit effort="1000.0" lower="-1.57075" upper="1.57075" velocity="1.0"/>
-    </joint>
-        <link name="pole">
-            <visual>
-            <geometry>
-                <cylinder length="0.3" radius="0.01"/>
-            </geometry>
-            <material name="black"/>
-            <origin rpy="0 0 0" xyz="0.0 0 -0.15"/>
-            </visual>
-        </link>
-        <joint name="pole_joint" type="revolute">
-            <origin xyz="-0.15 0 0.36" rpy="0 0 0"/>
-            <axis xyz="0 1 0"/>
-            <parent link="conector_pole"/>
-            <child link="pole"/>
-            <limit effort="1000.0" lower="-1.57075" upper="1.57075" velocity="1.0"/>
-        </joint>
-        <link name="pole_mass">
-            <visual>
-            <geometry>
-                <sphere radius="0.075"/>
-            </geometry>
-            <material name="blue"/>
-            <origin rpy="0 0 0" xyz="0.0 0 0.0"/>
-            </visual>
-        </link>
-        <joint name="pole_mass_joint" type="fixed">
-            <origin xyz="0 0 -1.5" rpy="0 0 0"/>
-            <axis xyz="0 0 0"/>
-            <parent link="pole"/>
-            <child link="pole_mass"/>
-        </joint>
-        <gazebo reference = "pole">
-            <material>Gazebo/Black</material>
-        </gazebo>
-        <gazebo reference = "pole_mass">
-            <material>Gazebo/Blue</material>
-        </gazebo>
-    <!--Pendulum/-->
     <!-- RIGHT WHEEL LINK 2-->
         <joint name="right_wheel_2_joint" type="continuous">

Commit message: pendulum correct

File: description/gazebo_control.xacro (robot description, xacro)
@@ -6,6 +6,4 @@
                 <left_joint>left_wheel_joint</left_joint>
                 <right_joint>right_wheel_joint</right_joint>
-                <!--left_joint>left_wheel_2_joint</left_joint>
-                <right_joint>right_wheel_2_joint</right_joint-->
                 <wheel_separation>0.35</wheel_separation>
                 <wheel_diameter>0.1</wheel_diameter>

File: description/pendulum.xacro (robot description, xacro)
@@ -2,85 +2,223 @@
 <robot xmlns:xacro="http://www.ros.org/wiki/xacro">
     <xacro:include filename="inertial_macros.xacro"/>
-        <!--Pendulum-->
-        <link name="conector_pole">
-            <inertial>
-                <origin xyz="0.0 0.0 0.0" rpy="0.0 0.0 0.0"/>
-                <mass value="0.01"/>
-                <inertia ixx="0.0" ixy="0.0" ixz="0.0" iyy="0.0" iyz="0.0" izz="0.0"/>
-            </inertial>
-            <visual>
-                <geometry>
-                    <box size="0.02 0.02 0.02"/>
-                </geometry>
-                <material name="black"/>
-                <origin rpy="0 0 0" xyz="0 0 0"/>
-            </visual>
-            <collision>
-                <geometry>
-                    <box size="0.02 0.02 0.02"/>
-                </geometry>
-            </collision>
-            <xacro:inertial_box mass="0.01" x="0.02" y="0.02" z="0.02">
-                <origin xyz="0 0 0" rpy="0 0 0"/>
-            </xacro:inertial_box>
-        </link>
-        <joint name="conector_pole_joint" type="fixed">
-            <parent link="chassis"/>
-            <child link="conector_pole"/>
-            <origin xyz="0.15 0 0.15" />
-        </joint>
-        <link name="pole">
-            <visual>
-                <geometry>
-                    <cylinder length="0.3" radius="0.01"/>
-                </geometry>
-                <material name="black"/>
-                <origin rpy="0 0 0" xyz="0 0 0"/>
-            </visual>
-            <collision>
-                <geometry>
-                    <cylinder length="0.3" radius="0.01"/>
-                </geometry>
-            </collision>
-            <xacro:inertial_cylinder mass="0.05"  radius="0.01" length="0.03">
-                <origin xyz="0 0 0" rpy="0 0 0"/>
-            </xacro:inertial_cylinder >
-        </link>
-        <joint name="pole_joint" type="revolute">
-            <parent link="conector_pole"/>
-            <child link="pole"/>
-            <origin xyz="0 0 0.3" rpy="0 0 0"/>
-            <axis xyz="0 1.0 0"/>
-            <limit effort="1000.0" lower="-0.57075" upper="0.57075" velocity="1.0"/>
-        </joint>
-            <!--link name="pole_mass">
-                <inertial>
-                    <origin xyz="0.0 0.0 0.0" rpy="0.0 0.0 0.0"/>
-                    <mass value="0.01"/>
-                    <inertia ixx="0.0" ixy="0.0" ixz="0.0" iyy="0.0" iyz="0.0" izz="0.0"/>
-                </inertial>
-                <visual>
-                <geometry>
-                    <sphere radius="0.075"/>
-                </geometry>
-                <material name="blue"/>
-                <origin rpy="0 0 0" xyz="0 0 0"/>
-                </visual>
-            </link>
-            <joint name="pole_mass_joint" type="fixed">
-                <origin xyz="0.15 0 1.5" rpy="0 0 0"/>
-                <axis xyz="0 0 0"/>
-                <parent link="pole"/>
-                <child link="pole_mass"/>
-            </joint-->
-            <gazebo reference = "pole">
-                <material>Gazebo/black</material>
-            </gazebo>
-            <gazebo reference = "conector_pole">
-                <material>Gazebo/white</material>
-            </gazebo>
-            <!--gazebo reference = "pole_mass">
-                <material>Gazebo/blue</material>
-            </gazebo-->
-        <!--Pendulum/-->
+         <!-- ######################################################################## /-->
+    <!--material color /-->
+    <material name="white">
+        <color rgba="1 1 1 1"/>
+    </material>
+    <material name="orange">
+        <color rgba="1 0.3 0.1 1"/>
+    </material>
+    <material name="blue">
+        <color rgba="0.2 0.2 1 1"/>
+    </material>
+    <material name="black">
+        <color rgba="0 0 0 1"/>
+    </material>
+    <material name="red">
+        <color rgba="1 0 0 1"/>
+    </material>
+    <gazebo>
+        <plugin filename="libgazebo_ros_control.so" name="gazebo_ros_control">
+          <robotSimType>sr_gazebo_sim/SrGazeboHWSim</robotSimType>
+        </plugin>
+      </gazebo>
+    <!-- BASE LINK/-->
+    <link name="base_link">
+    </link>
+    <!-- BASE LINK-->
+    <!-- ########################################################################-->
+    <!--CHASSIS LINK/-->
+    <joint name="chassis_joint" type="fixed">
+        <parent link="base_link"/>
+        <child link="chassis"/>
+        <origin xyz="0.0 0.0 0.0"/>
+    </joint>
+    <link name="chassis">
+        <visual>
+            <origin xyz="0.0 0.0 0.075"/>
+            <geometry>
+                <box size="0.3 0.3 0.15"/>
+            </geometry>
+            <material name="blue"/>
+        </visual>
+        <collision>
+            <origin xyz="0.0 0.0 0.075"/>
+            <geometry>
+                <box size="0.3 0.3 0.15"/>
+            </geometry>
+        </collision>
+        <xacro:inertial_box mass="1.5" x="0.3" y="0.3" z="0.15">
+            <origin xyz="0.0 0.0 0.075" rpy="0.0 0.0 0.0"/>
+        </xacro:inertial_box>
+    </link>
+    <gazebo reference = "chassis">
+        <material>Gazebo/Blue</material>
+    </gazebo>
+    <!--CHASSIS LINK-->
+    <!-- ######################################################################## -->
+    <!-- LEFT WHEEL LINK -->
+    <joint name="left_wheel_joint" type="continuous">
+            <parent link="base_link"/>
+            <child link="left_wheel"/>
+            <origin xyz="-0.1 -0.175 0.0" rpy="-${pi/2}  0.0 0.0"/>
+            <axis xyz="0.0 0.0 -1.0"/>
+    </joint>
+    <link name="left_wheel">
+        <visual>
+            <origin xyz="0.0 0.0 0.0" rpy="0.0  0.0 0.0"/>
+            <geometry>
+                <cylinder radius="0.05" length="0.04"/>
+            </geometry>
+            <material name="white"/>
+        </visual>
+        <collision>
+            <geometry>
+                <cylinder radius="0.05" length="0.04"/>
+            </geometry>
+        </collision>
+        <xacro:inertial_cylinder mass="0.15"  radius="0.05" length="0.04">
+            <origin xyz="0.0 0.0 0.0" rpy="0.0 0.0 0.0"/>
+        </xacro:inertial_cylinder >
+    </link>
+    <gazebo reference = "left_wheel">
+        <material>Gazebo/White</material>
+    </gazebo>
+    <!-- LEFT WHEEL LINK -->
+    <!-- ######################################################################## -->
+    <!-- RIGHT WHEEL LINK -->
+    <joint name="right_wheel_joint" type="continuous">
+            <parent link="base_link"/>
+            <child link="right_wheel"/>
+            <origin xyz="-0.1 0.175 0.0" rpy="${pi/2}  0.0 0.0"/>
+            <axis xyz="0.0 0.0 1.0"/>
+    </joint>
+    <link name="right_wheel">
+        <visual>
+            <origin xyz="0.0 0.0 0.0" rpy="0.0 0.0 0.0"/>
+            <geometry>
+                <cylinder radius="0.05" length="0.04"/>
+            </geometry>
+            <material name="white"/>
+        </visual>
+        <collision>
+            <geometry>
+                <cylinder radius="0.05" length="0.04"/>
+            </geometry>
+        </collision>
+        <xacro:inertial_cylinder mass="0.15" length="0.04" radius="0.05" >
+            <origin xyz="0.0 0.0 0.0" rpy="0.0 0.0 0.0"/>
+        </xacro:inertial_cylinder >
+    </link>
+    <gazebo reference = "right_wheel">
+        <material>Gazebo/White</material>
+    </gazebo>
+     <!-- RIGHT WHEEL LINK -->
+    <!-- ######################################################################## -->
+    <!-- CASTER WHEEL LINK-->
+    <joint name="left_wheel_2_joint" type="continuous">
+        <parent link="base_link"/>
+        <child link="left_wheel_2"/>
+        <origin xyz="0.1 -0.175 0.0" rpy="-${pi/2}  0.0 0.0"/>
+        <axis xyz="0.0 0.0 -1.0"/>
+    </joint>
+    <link name="left_wheel_2">
+        <visual>
+            <origin xyz="0.0 0.0 0.0" rpy="0.0  0.0 0.0"/>
+            <geometry>
+                <cylinder radius="0.05" length="0.04"/>
+            </geometry>
+            <material name="white"/>
+        </visual>
+        <collision>
+            <geometry>
+                <cylinder radius="0.05" length="0.04"/>
+            </geometry>
+        </collision>
+        <xacro:inertial_cylinder mass="0.15"  radius="0.05" length="0.04">
+            <origin xyz="0.0 0.0 0.0" rpy="0.0 0.0 0.0"/>
+        </xacro:inertial_cylinder >
+    </link>
+    <gazebo reference = "left_wheel_2">
+        <material>Gazebo/White</material>
+    </gazebo>
+<!-- RIGHT WHEEL LINK -->
+    <joint name="right_wheel_2_joint" type="continuous">
+            <parent link="base_link"/>
+            <child link="right_wheel_2"/>
+            <origin xyz="0.1 0.175 0.0" rpy="${pi/2}  0.0 0.0"/>
+            <axis xyz="0.0 0.0 1.0"/>
+    </joint>
+    <link name="right_wheel_2">
+        <visual>
+            <origin xyz="0.0 0.0 0.0" rpy="0.0 0.0 0.0"/>
+            <geometry>
+                <cylinder radius="0.05" length="0.04"/>
+            </geometry>
+            <material name="white"/>
+        </visual>
+        <collision>
+            <geometry>
+                <cylinder radius="0.05" length="0.04"/>
+            </geometry>
+        </collision>
+        <xacro:inertial_cylinder mass="0.15" length="0.04" radius="0.05" >
+            <origin xyz="0.0 0.0 0.0" rpy="0.0 0.0 0.0"/>
+        </xacro:inertial_cylinder >
+    </link>
+    <gazebo reference = "right_wheel_2">
+        <material>Gazebo/White</material>
+    </gazebo>
+    <link name="pole">
+        <visual>
+            <geometry>
+                <cylinder length="0.3" radius="0.01"/>
+            </geometry>
+            <material name="orange"/>
+            <origin rpy="0.0 0.0 -0.15" xyz="0.0 0.0 0.3"/>
+        </visual>
+        <collision>
+            <geometry>
+                <cylinder length="0.3" radius="0.01"/>
+            </geometry>
+        </collision>
+        <xacro:inertial_cylinder mass="0.0"  radius="0.01" length="0.03">
+            <origin xyz="0.0 0.0 0.0" rpy="0.0 0.0 0.0"/>
+        </xacro:inertial_cylinder >
+    </link>
+    <joint name="pole_joint" type="revolute">
+        <parent link="chassis"/>
+        <child link="pole"/>
+        <origin xyz="0.0 0.0 0.0" rpy="0.0 0.0 0.0"/>
+        <axis xyz="0.0 1.0 0.0"/>
+        <limit effort="1000.0" lower="-0.78" upper="0.78" velocity="1.0"/>
+    </joint>
+    <link name="conector_pole">
+        <visual>
+            <geometry>
+                <box size="0.02 0.02 0.02"/>
+            </geometry>
+            <material name="black"/>
+            <origin rpy="0.0 0.0 0.0" xyz="0.0 0.0 0.0"/>
+        </visual>
+        <collision>
+            <geometry>
+                <box size="0.02 0.02 0.02"/>
+            </geometry>
+        </collision>
+        <xacro:inertial_box mass="0.0" x="0.02" y="0.02" z="0.02">
+            <origin xyz="0.0 0.0 0.0" rpy="0.0 0.0 0.0"/>
+        </xacro:inertial_box>
+    </link>
+    <joint name="conector_pole_joint" type="fixed">
+        <parent link="pole"/>
+        <child link="conector_pole"/>
+        <origin xyz="0.0 0.0 0.45" />
+    </joint>
+    <gazebo reference = "pole">
+        <material>Gazebo/Orange</material>
+    </gazebo>
+    <gazebo reference = "conector_pole">
+        <material>Gazebo/Black</material>
+    </gazebo>
 </robot>

File: description/robot.urdf.xacro (robot description, xacro)
@@ -2,8 +2,8 @@
 <robot xmlns:xacro="http://www.ros.org/wiki/xacro"  name="robot">
     <xacro:include filename = "robot_core.xacro"/>
-    <!--xacro:include filename = "robot_core_2.xacro"/-->
+    <xacro:include filename = "robot_core_2.xacro"/>
     <xacro:include filename = "gazebo_control.xacro"/>
-    <xacro:include filename = "pendulum.xacro"/>
+    <!--xacro:include filename = "pendulum.xacro"/-->
     <!--xacro:include filename = "lidar.xacro"/-->
-    <xacro:include filename = "camera.xacro"/>
+    <!--xacro:include filename = "camera.xacro"/-->
 </robot>

File: description/robot_core.xacro (robot description, xacro)
@@ -33,9 +33,9 @@
         <parent link="base_link"/>
         <child link="chassis"/>
-        <origin xyz="-0.1 0 0"/>
+        <origin xyz="0.0 0.0 0.0"/>
     </joint>
     <link name="chassis">
         <visual>
-            <origin xyz="0.15 0 0.075"/>
+            <origin xyz="0.0 0.0 0.075"/>
             <geometry>
                 <box size="0.3 0.3 0.15"/>
@@ -44,11 +44,11 @@
         </visual>
         <collision>
-            <origin xyz="0.15 0 0.075"/>
+            <origin xyz="0.0 0.0 0.075"/>
             <geometry>
                 <box size="0.3 0.3 0.15"/>
             </geometry>
         </collision>
-        <xacro:inertial_box mass="0.5" x="0.3" y="0.3" z="0.15">
-            <origin xyz="0.15 0 0.075" rpy="0 0 0"/>
+        <xacro:inertial_box mass="1.5" x="0.3" y="0.3" z="0.15">
+            <origin xyz="0.0 0.0 0.075" rpy="0.0 0.0 0.0"/>
         </xacro:inertial_box>
     </link>
@@ -62,9 +62,10 @@
             <parent link="base_link"/>
             <child link="left_wheel"/>
-            <origin xyz="0.14 0.175 0" rpy="-${pi/2} 0 0"/>
-            <axis xyz="0 0 1"/>
+            <origin xyz="-0.1 -0.175 0.0" rpy="-${pi/2}  0.0 0.0"/>
+            <axis xyz="0.0 0.0 -1.0"/>
     </joint>
     <link name="left_wheel">
         <visual>
+            <origin xyz="0.0 0.0 0.0" rpy="0.0  0.0 0.0"/>
             <geometry>
                 <cylinder radius="0.05" length="0.04"/>
@@ -77,6 +78,6 @@
             </geometry>
         </collision>
-        <xacro:inertial_cylinder mass="0.1"  radius="0.05" length="0.04">
-            <origin xyz="0 0 0" rpy="0 0 0"/>
+        <xacro:inertial_cylinder mass="0.15"  radius="0.05" length="0.04">
+            <origin xyz="0.0 0.0 0.0" rpy="0.0 0.0 0.0"/>
         </xacro:inertial_cylinder >
     </link>
@@ -90,9 +91,10 @@
             <parent link="base_link"/>
             <child link="right_wheel"/>
-            <origin xyz="0.14 -0.175 0" rpy="${pi/2} 0 0"/>
-            <axis xyz="0 0 -1"/>
+            <origin xyz="-0.1 0.175 0.0" rpy="${pi/2}  0.0 0.0"/>
+            <axis xyz="0.0 0.0 1.0"/>
     </joint>
     <link name="right_wheel">
         <visual>
+            <origin xyz="0.0 0.0 0.0" rpy="0.0 0.0 0.0"/>
             <geometry>
                 <cylinder radius="0.05" length="0.04"/>
@@ -105,6 +107,6 @@
             </geometry>
         </collision>
-        <xacro:inertial_cylinder mass="0.1" length="0.04" radius="0.05" >
-            <origin xyz="0 0 0" rpy="0 0 0"/>
+        <xacro:inertial_cylinder mass="0.15" length="0.04" radius="0.05" >
+            <origin xyz="0.0 0.0 0.0" rpy="0.0 0.0 0.0"/>
         </xacro:inertial_cylinder >
     </link>
@@ -118,5 +120,5 @@
         <parent link="chassis"/>
         <child link="caster_wheel"/>
-        <origin xyz="0.08 0 0"/>
+        <origin xyz="0.08 0.0 0.0"/>
     </joint>
     <link name="caster_wheel">
@@ -132,6 +134,6 @@
             </geometry>
         </collision>
-        <xacro:inertial_sphere mass="0.1" radius="0.05" >
-            <origin xyz="0 0 0" rpy="0 0 0"/>
+        <xacro:inertial_sphere mass="0.3" radius="0.05" >
+            <origin xyz="0.0 0.0 0.0" rpy="0.0 0.0 0.0"/>
         </xacro:inertial_sphere>
     </link>
@@ -141,4 +143,3 @@
         <mu2 value = "0.001"/>
     </gazebo>
-    <!-- CASTER WHEEL LINK-->
 </robot>
