Commit message: new files

File: description/gazebo_control.xacro (robot description, xacro)
@@ -8,13 +8,16 @@
                 <wheel_separation>0.35</wheel_separation>
                 <wheel_diameter>0.1</wheel_diameter>
+            <!-- Connector inf -->
+                <element2_link_joint>element2_link_joint</element2_link_joint>
             <!-- limits -->
-            <max_wheel_torque>200</max_wheel_torque>
-            <max_acceleration>10.0</max_acceleration>
+                <max_wheel_torque>200</max_wheel_torque>
+                <max_acceleration>10.0</max_acceleration>
             <!-- Output -->
-            <odometry_frame>odom</odometry_frame>
-            <robot_base_frame>base_link</robot_base_frame>
-            <publish_odom>true</publish_odom>
-            <publish_odom_tf>true</publish_odom_tf>
-            <publish_wheel_tf>true</publish_wheel_tf>
+                <odometry_frame>odom</odometry_frame>
+                <robot_base_frame>base_link</robot_base_frame>
+                <robot_base_frame_2>base_link_2</robot_base_frame_2>
+                <publish_odom>true</publish_odom>
+                <publish_odom_tf>true</publish_odom_tf>
+                <publish_wheel_tf>true</publish_wheel_tf>
         </plugin>
     </gazebo>

File: description/robot.urdf.xacro (robot description, xacro)
@@ -1,5 +1,4 @@
 <?xml version="1.0"?>
 <robot xmlns:xacro="http://www.ros.org/wiki/xacro"  name="robot">
-    <xacro:include filename = "color.xacro"/>
     <xacro:include filename = "robot_core.xacro"/>
     <!--xacro:include filename = "robot_core_2.xacro"/-->

File: description/robot_core.xacro (robot description, xacro)
@@ -2,9 +2,24 @@
 <robot xmlns:xacro="http://www.ros.org/wiki/xacro">
     <xacro:include filename="inertial_macros.xacro"/>
+    <material name="white">
+        <color rgba="1 1 1 1"/>
+    </material>
+    <material name="orange">
+        <color rgba="1 0.3 0.1 1"/>
+    </material>
+    <material name="blue">
+        <color rgba="0.2 0.2 1 1"/>
+    </material>
+    <material name="black">
+        <color rgba="0 0 0 1"/>
+    </material>
+    <material name="red">
+        <color rgba="1 0 0 1"/>
+    </material>
     <gazebo>
         <plugin filename="libgazebo_ros_control.so" name="gazebo_ros_control">
           <robotSimType>sr_gazebo_sim/SrGazeboHWSim</robotSimType>
         </plugin>
-      </gazebo>
+    </gazebo>
     <!-- BASE LINK/-->
     <link name="base_link">

File: description/robot_core_2.xacro (robot description, xacro)
@@ -2,73 +2,81 @@
 <robot xmlns:xacro="http://www.ros.org/wiki/xacro">
     <xacro:include filename="inertial_macros.xacro"/>
-    <!--Connector-->
-    <joint name="conector_joint" type="fixed">
+    <joint name="element_link_joint" type="fixed">
+        <axis xyz="1 0 0"/>
         <parent link="chassis"/>
-        <child link="conector_link"/>
-        <origin xyz="-0.005 0 0.05" rpy="0 0 0"/>
+        <child link="element_link"/>
+        <origin xyz="-0.075 0 0.06" rpy="0 0 0"/>
     </joint>
-    <link name="conector_link">
+    <link name="element_link">
         <visual>
+            <origin xyz="0 0 0" rpy="0 0 0"/>
             <geometry>
-                <box size="0.01 0.03 0.03"/>
+                <box size="0.15 0.02 0.02"/>
             </geometry>
             <material name="red"/>
         </visual>
         <collision>
-            <box size="0.01 0.03 0.03"/>
+            <origin xyz="0 0 0" rpy="0 0 0"/>
+            <geometry>
+                <box size="0.15 0.02 0.02"/>
+            </geometry>
         </collision>
-        <xacro:inertial_box mass="0.01" x="0.01" y="0.03" z="0.03">
-            <origin xyz="0.15 0 0.075" rpy="0 0 0"/>
-        </xacro:inertial_box>
-    </link>
-    <gazebo reference="conector_link">
-        <material>Gazebo/Red</material>
-    </gazebo>
-    <!--element1-->
-    <joint name="element1_joint" type="fixed">
-        <origin xyz="0 0 0" rpy="0 0 0"/>
-        <axis xyz="1 0 0"/>
-        <parent link="conector_link"/>
-        <child link="element1_link"/>
-    </joint>
-    <link name="element1_link">
-        <visual>
-            <geometry>
-                <box size="0.3 0.02 0.02"/>
-            </geometry>
-            <material name="red"/>
-        </visual>
-        <collision>
-            <box size="0.3 0.02 0.02"/>
-        </collision>
-        <xacro:inertial_box mass="0.1" x="0.3" y="0.02" z="0.02">
+        <xacro:inertial_box mass="0.0001" x="0.3" y="0.02" z="0.02">
             <origin xyz="0 0 0" rpy="0 0 0"/>
         </xacro:inertial_box>
     </link>
-    <gazebo reference="element1_link">
+    <gazebo reference="element_link">
         <material>Gazebo/Red</material>
     </gazebo>
+        <joint name="conector_joint" type="revolute">
+                <parent link="element_link"/>
+                <child link="conector_link"/>
+                <axis xyz="0 0 1"/>
+                <limit effort="1000.0" lower="-1.5708" upper="1.5708" velocity="0.5"/>
+                <origin xyz="-0.075 0 0" rpy="0 0 0"/>
+        </joint>
+        <link name="conector_link">
+            <visual>
+                <origin xyz="0 0 0" rpy="0 0 0"/>
+                <geometry>
+                    <box size="0.03 0.03 0.03"/>
+                </geometry>
+                <material name="black"/>
+            </visual>
+            <collision>
+                <origin xyz="0 0 0" rpy="0 0 0"/>
+                <geometry>
+                    <box size="0.03 0.03 0.03"/>
+                </geometry>
+            </collision>
+            <xacro:inertial_box mass="0.0001" x="0.01" y="0.03" z="0.03">
+                <origin xyz="0 0 0" rpy="0 0 0"/>
+            </xacro:inertial_box>
+        </link>
+        <gazebo reference="conector_link">
+            <material>Gazebo/Black</material>
+        </gazebo>
     <!--element2/-->
-        <joint name="element2_joint" type="revolute">
-            <parent link="element1_link"/>
+        <joint name="element2_link_joint" type="fixed">
+            <parent link="conector_link"/>
             <child link="element2_link"/>
-            <axis xyz="0 0 1"/>
-            <!--limit effort="1000.0" lower="0.0" upper="0.548" velocity="0.5"/-->
-            <origin xyz="-0.15 0 0" rpy="0 0 0"/>
+            <origin xyz="0 0 0" rpy="0 0 0"/>
         </joint>
         <link name="element2_link">
             <visual>
+                <origin xyz="-0.075 0 0" rpy="0 0 0"/>
                 <geometry>
                     <box size="0.15 0.02 0.02"/>
                 </geometry>
-                <origin rpy="1.57074 0 0" xyz="0.075 0 0"/>>
                 <material name="red"/>
             </visual>
             <collision>
-                <origin xyz="0.0 0.0 0.0" rpy="0.0 0.0 0.0"/>
-                <box size="0.15 0.02 0.02"/>
+                <origin xyz="-0.075 0 0" rpy="0 0 0"/>
+                <geometry>
+                    <box size="0.15 0.02 0.02"/>
+                </geometry>
             </collision>
-            <xacro:inertial_box mass="0.01" x="0.15" y="0.02" z="0.02">
-                <origin xyz="0 0 0" rpy="0 0 0"/>
+            <xacro:inertial_box mass="0.0001" x="0.15" y="0.02" z="0.02">
+                <origin xyz="-0.075 0 0" rpy="0 0 0"/>
             </xacro:inertial_box>
         </link>
@@ -76,37 +84,12 @@
             <material>Gazebo/Red</material>
         </gazebo>
-    <!--conector_2/-->
-        <joint name="conector_2_joint" type="fixed">
-                <parent link="element2_link"/>
-                <child link="conector_2_link"/>
-                <origin xyz="-0.075 0 0" rpy="0 0 0"/>
-        </joint>
-        <link name="conector_2_link">
-            <visual>
-                <geometry>
-                    <box size="0.01 0.03 0.03"/>
-                </geometry>
-                <material name="red"/>
-            </visual>
-            <collision>
-                <origin xyz="0.0 0.0 0.0" rpy="0.0 0.0 0.0"/>
-                <box size="0.01 0.03 0.03"/>
-            </collision>
-            <xacro:inertial_box mass="0.01" x="0.01" y="0.03" z="0.03">
-                <origin xyz="0 0 0" rpy="0 0 0"/>
-            </xacro:inertial_box>
-        </link>
-        <gazebo reference="conector_2_link">
-            <material>Gazebo/Red</material>
-        </gazebo>
-    <!--CHASSIS LINK 2-->
-        <joint name="chassis_2_joint" type="fixed">
-            <parent link="conector_2_link"/>
+        <!--joint name="chassis_2_joint" type="fixed">
+            <parent link="element2_link"/>
             <child link="chassis_2"/>
-            <origin xyz="0 0 -0.05"/>
+            <origin xyz="0 0 0" rpy="0 0 0"/>
         </joint>
         <link name="chassis_2">
             <visual>
-                <origin xyz="0 0 0"/>
+                <origin xyz="-0.2 0 0.02" rpy="0 0 0"/>
                 <geometry>
                     <box size="0.3 0.3 0.15"/>
@@ -115,11 +98,11 @@
             </visual>
             <collision>
-                <origin xyz="0 0 0"/>
+                <origin xyz="-0.2 0 0.02" rpy="0 0 0"/>
                 <geometry>
                     <box size="0.3 0.3 0.15"/>
                 </geometry>
             </collision>
-            <xacro:inertial_box mass="0.5" x="0.3" y="0.3" z="0.15">
-                <origin xyz="0 0 0" rpy="0 0 0"/>
+            <xacro:inertial_box mass="0.3" x="0.3" y="0.3" z="0.15">
+                <origin xyz="-0.2 0 0.02" rpy="0 0 0"/>
             </xacro:inertial_box>
         </link>
@@ -127,13 +110,13 @@
             <material>Gazebo/Blue</material>
         </gazebo>
-    <!-- LEFT WHEEL LINK 2-->
-        <joint name="left_wheel_2_joint" type="fixed">
+        <joint name="left_wheel_2_joint" type="continuous">
                 <parent link="chassis_2"/>
                 <child link="left_wheel_2"/>
-                <origin xyz="-0.06 0.175 0" rpy="-${pi/2} 0 0"/>
+                <origin xyz="-0.1 0.175 -0.075" rpy="-${pi/2} 0 0"/>
                 <axis xyz="0 0 1"/>
         </joint>
         <link name="left_wheel_2">
             <visual>
+                <origin xyz="0 0 0" rpy="0 0 0"/>
                 <geometry>
                     <cylinder radius="0.05" length="0.04"/>
@@ -142,4 +125,5 @@
             </visual>
             <collision>
+                <origin xyz="0 0 0" rpy="0 0 0"/>
                 <geometry>
                     <cylinder radius="0.05" length="0.04"/>
@@ -153,13 +137,13 @@
             <material>Gazebo/White</material>
         </gazebo>
-    <!-- RIGHT WHEEL LINK 2-->
         <joint name="right_wheel_2_joint" type="continuous">
                 <parent link="chassis_2"/>
                 <child link="right_wheel_2"/>
-                <origin xyz="-0.06 -0.175 0" rpy="${pi/2} 0 0"/>
+                <origin xyz="-0.1 -0.175 -0.075" rpy="${pi/2} 0 0"/>
                 <axis xyz="0 0 -1"/>
         </joint>
         <link name="right_wheel_2">
             <visual>
+                <origin xyz="0 0 0" rpy="0 0 0"/>
                 <geometry>
                     <cylinder radius="0.05" length="0.04"/>
@@ -168,9 +152,10 @@
             </visual>
             <collision>
+                <origin xyz="0 0 0" rpy="0 0 0"/>
                 <geometry>
                     <cylinder radius="0.05" length="0.04"/>
                 </geometry>
             </collision>
-            <xacro:inertial_cylinder mass="0.1" length="0.04" radius="0.05" >
+            <xacro:inertial_cylinder mass="0.1"  radius="0.05" length="0.04">
                 <origin xyz="0 0 0" rpy="0 0 0"/>
             </xacro:inertial_cylinder >
@@ -179,12 +164,12 @@
             <material>Gazebo/White</material>
         </gazebo>
-    <!-- CASTER WHEEL LINK-->
-        <joint name="caster_wheel_2_joint" type="fixed">
+        <!joint name="caster_wheel_2_joint" type="fixed">
             <parent link="chassis_2"/>
             <child link="caster_wheel_2"/>
-            <origin xyz="-0.25 0 0"/>
+            <origin xyz="0.1 0 -0.075" rpy="0 0 0"/>
         </joint>
         <link name="caster_wheel_2">
             <visual>
+                <origin xyz="0 0 0" rpy="0 0 0"/>
                 <geometry>
                     <sphere radius="0.05"/>
@@ -193,4 +178,5 @@
             </visual>
             <collision>
+                <origin xyz="0 0 0" rpy="0 0 0"/>
                 <geometry>
                     <sphere radius="0.05"/>
@@ -205,4 +191,4 @@
             <mu1 value = "0.001"/>
             <mu2 value = "0.001"/>
-        </gazebo>
+        </gazebo-->
 </robot>
